Commit message: perf<diffbot urdf>: 提升模型美观性

File: description/urdf/diffbot_description.urdf.xacro (robot description, xacro)
@@ -10,10 +10,10 @@
     <xacro:property name="wheel_mass" value="0.3" /> <!-- arbitrary value for wheel mass -->
     <xacro:property name="wheel_len" value="0.1" />
-    <xacro:property name="wheel_radius" value="0.3" />
-    <xacro:property name="caster_wheel_mass" value="0.1" /> <!-- arbitrary value for caster wheel
-    mass -->
+    <xacro:property name="wheel_radius" value="0.5" />
+    <xacro:property name="wheel_separation" value="${base_width/2 + wheel_len/2 + 0.02}" />
+    <xacro:property name="caster_wheel_mass" value="0.1" /> <!-- arbitrary value for caster wheel mass -->
     <xacro:property name="caster_wheel_radius" value="0.3" />
-    <xacro:property name="z_offset" value="-${base_height/2}" /> <!-- Space btw top of beam and the
-    each joint -->
+    <xacro:property name="caster_offset" value="0.2"/>
+    <xacro:property name="z_offset" value="${wheel_radius - caster_wheel_radius - caster_offset}" /> <!-- Space btw top of beam and the each joint -->
     <!-- Base Link -->
     <link name="${prefix}base_link">
@@ -44,5 +44,5 @@
       <parent link="${prefix}base_link" />
       <child link="${prefix}left_wheel" />
-      <origin xyz="0 ${base_width/2} ${z_offset}" rpy="0 0 0" />
+      <origin xyz="0 ${wheel_separation} ${z_offset}" rpy="0 0 0" />
       <axis xyz="0 1 0" />
       <dynamics damping="0.2" />
@@ -77,5 +77,5 @@
       <parent link="${prefix}base_link" />
       <child link="${prefix}right_wheel" />
-      <origin xyz="0 -${base_width/2} ${z_offset}" rpy="0 0 0" />
+      <origin xyz="0 -${wheel_separation} ${z_offset}" rpy="0 0 0" />
       <axis xyz="0 1 0" />
       <dynamics damping="0.2" />
@@ -110,5 +110,5 @@
       <parent link="${prefix}base_link" />
       <child link="${prefix}caster_frontal_wheel" />
-      <origin xyz="${base_width/2 - caster_wheel_radius} 0 ${z_offset}" rpy="0 0 0" />
+      <origin xyz="${base_width/2 - caster_wheel_radius} 0 -${caster_offset}" rpy="0 0 0" />
     </joint>
     <!-- caster frontal wheel Link -->
@@ -140,5 +140,5 @@
       <parent link="${prefix}base_link" />
       <child link="${prefix}caster_rear_wheel" />
-      <origin xyz="${-base_width/2 + caster_wheel_radius} 0 ${z_offset}" rpy="0 0 0" />
+      <origin xyz="${-base_width/2 + caster_wheel_radius} 0 -${caster_offset}" rpy="0 0 0" />
     </joint>
     <!-- caster rear wheel Link -->

Commit message: perf<gazebo>: 提升小车运行速度

File: description/urdf/diffbot_description.urdf.xacro (robot description, xacro)
@@ -47,5 +47,4 @@
       <axis xyz="0 1 0" />
       <dynamics damping="0.2" />
-      <limit effort="100" velocity="1.0" />
     </joint>
     <!-- left wheel Link -->
@@ -80,5 +79,4 @@
       <axis xyz="0 1 0" />
       <dynamics damping="0.2" />
-      <limit effort="100" velocity="1.0" />
     </joint>
     <!-- right wheel Link -->
