Commit message: fix<mini_4wd/urdf>: 修复资源文件路径配置问题

File: models/mini_4wd/urdf/all.xacro (robot description, xacro)
@@ -25,6 +25,6 @@
   <xacro:property name="box_width" value="0.1" />
   <xacro:property name="box_mass" value="0.6" />
-  <xacro:property name="urdf_dir" value="$(find ugv_ctrl)/description/mini_4wd/urdf" />
-  <xacro:property name="mesh_dir" value="package://ugv_ctrl/description/mini_4wd/meshes" />
+  <xacro:property name="urdf_dir" value="$(find ugv_ctrl)/models/mini_4wd/urdf" />
+  <xacro:property name="mesh_dir" value="package://ugv_ctrl/models/mini_4wd/meshes" />
   <xacro:macro name="box_inertial_matrix" params="m w h d">
     <inertial>

Commit message: fix<mini_4wd/ros2_control>: 修复 ros2 control 配置

File: models/mini_4wd/urdf/all.xacro (robot description, xacro)
@@ -25,5 +25,7 @@
   <xacro:property name="box_width" value="0.1" />
   <xacro:property name="box_mass" value="0.6" />
-  <xacro:property name="urdf_dir" value="$(find ugv_ctrl)/models/mini_4wd/urdf" />
+  <xacro:property name="model_name" value="mini_4wd" />
+  <xacro:property name="model_dir" value="$(find ugv_ctrl)/models/${model_name}" />
+  <xacro:property name="urdf_dir" value="${model_dir}/urdf" />
   <xacro:property name="mesh_dir" value="package://ugv_ctrl/models/mini_4wd/meshes" />
   <xacro:macro name="box_inertial_matrix" params="m w h d">

File: models/mini_4wd/urdf/gazebo.xacro (robot description, xacro)
@@ -4,5 +4,5 @@
     <plugin filename="gz_ros2_control-system"
       name="gz_ros2_control::GazeboSimROS2ControlPlugin">
-      <parameters>$(find ugv_ctrl)/config/diffbot_controllers.yaml</parameters>
+      <parameters>${model_dir}/control_cfg.yml</parameters>
     </plugin>
     <plugin

Commit message: fix<mini_4wd/urdf>: 更新小车尺寸

File: models/mini_4wd/urdf/all.xacro (robot description, xacro)
@@ -21,7 +21,7 @@
   <xacro:property name="box_position_y" value="0" />
   <xacro:property name="box_position_z" value="0.07" />
-  <xacro:property name="box_length" value="0.18" />
-  <xacro:property name="box_height" value="0.04" />
-  <xacro:property name="box_width" value="0.1" />
+  <xacro:property name="box_length" value="0.27" />
+  <xacro:property name="box_width" value="0.19" />
+  <xacro:property name="box_height" value="0.075" />
   <xacro:property name="box_mass" value="0.6" />
   <xacro:property name="model_name" value="mini_4wd" />
