Commit message: fix<mini_4wd/urdf/body>: 修复车体碰撞体积

File: models/mini_4wd/urdf/body.xacro (robot description, xacro)
@@ -15,5 +15,5 @@
     </visual>
     <collision>
-      <origin xyz="0 0 0" rpy="0 0 0" />
+      <origin xyz="${box_position_x} ${box_position_y} ${box_position_z}" rpy="0 0 0" />
       <geometry>
         <!-- <mesh filename="${mesh_dir}/base_link.STL" /> -->
