Commit message: fix<mini_4wd>: 修复标签cylinder属性

File: models/mini_4wd/urdf/wheels.xacro (robot description, xacro)
@@ -17,8 +17,5 @@
         <geometry>
           <!-- <mesh filename="${mesh_dir}/${mesh_name}.STL" /> -->
-          <cylinder>
-            <radius>0.033</radius>
-            <length>0.035</length>
-          </cylinder>
+          <cylinder radius="0.033" length="0.035" />
         </geometry>
       </collision>

Commit message: fix<mini_4wd/urdf/wheel>: 修复车轮碰撞体积

File: models/mini_4wd/urdf/wheels.xacro (robot description, xacro)
@@ -5,4 +5,5 @@
         link_name
         mesh_name
+        xyz_offset
         *origin *mass *inertia">
     <link name="${link_name}">
@@ -14,8 +15,7 @@
       </visual>
       <collision>
-        <origin xyz="0 0 0" rpy="0 0 0" />
+        <origin xyz="${xyz_offset}" rpy="${M_PI/2} 0 0" />
         <geometry>
-          <!-- <mesh filename="${mesh_dir}/${mesh_name}.STL" /> -->
-          <cylinder radius="0.033" length="0.035" />
+          <cylinder radius="0.035" length="0.009" />
         </geometry>
       </collision>
@@ -42,5 +42,6 @@
   <xacro:create_wheel_link
     link_name="$(arg prefix)right_front_wheel_link"
-    mesh_name="right_front_wheel_link">
+    mesh_name="right_front_wheel_link"
+    xyz_offset="0 -0.021 0">
     <origin xyz="6.832E-08 -0.0098111 -7.0676E-07" rpy="0 0 0" />
     <mass value="${wheel_mass}" />
@@ -55,5 +56,6 @@
   <xacro:create_wheel_link
     link_name="$(arg prefix)left_front_wheel_link"
-    mesh_name="left_front_wheel_link">
+    mesh_name="left_front_wheel_link"
+    xyz_offset="0 0.021 0">
     <origin xyz="-6.8329E-08 0.0098111 -7.0684E-07" rpy="0 0 0" />
     <mass value="${wheel_mass}" />
@@ -68,5 +70,6 @@
   <xacro:create_wheel_link
     link_name="$(arg prefix)right_rear_wheel_link"
-    mesh_name="right_rear_wheel_link">
+    mesh_name="right_rear_wheel_link"
+    xyz_offset="0 -0.021 0">
     <origin xyz="6.832E-08 -0.0098111 -7.0676E-07" rpy="0 0 0" />
     <mass value="${wheel_mass}" />
@@ -81,5 +84,6 @@
   <xacro:create_wheel_link
     link_name="$(arg prefix)left_rear_wheel_link"
-    mesh_name="left_rear_wheel_link">
+    mesh_name="left_rear_wheel_link"
+    xyz_offset="0 0.021 0">
     <origin xyz="-6.8366E-08 0.0098111 -7.068E-07" rpy="0 0 0" />
     <mass value="${wheel_mass}" />
