Commit message: fix<min_4wd/urdf>: 修复传感器碰撞体积

File: models/mini_4wd/urdf/camera.xacro (robot description, xacro)
@@ -6,12 +6,10 @@
       <origin xyz="0 0 0" rpy="0 0 0 " />
       <geometry>
-        <mesh
-          filename="${mesh_dir}/camera_link.DAE" />
+        <mesh filename="${mesh_dir}/camera_link.DAE" />
       </geometry>
     </visual>
     <collision>
-      <origin xyz="0 0 0" rpy="0 0 0 " />
+      <origin xyz="0 0 0" rpy="0 0 0" />
       <geometry>
-        <!-- <mesh filename="${mesh_dir}/camera_link.STL" /> -->
         <box size="0.046 0.165 0.077" />
       </geometry>

File: models/mini_4wd/urdf/laser.xacro (robot description, xacro)
@@ -11,7 +11,6 @@
     </visual>
     <collision>
-      <origin xyz="0 0 0" rpy="0 0 0" />
+      <origin xyz=" 0 0 0 " rpy="0 0 0" />
       <geometry>
-        <!-- <mesh filename="${mesh_dir}/laser_link.STL" /> -->
         <box size="0.1 0.074 0.078" />
       </geometry>
